File: Analysis/Collection/Node/Hardware/Node.sch (EAGLE design)
At the start: 27 parts, among them IC1 4050D, IC2 LP298XS, IC3 DS3231/SO, M2 WIRELESS-NRF24L01-PA-EXT, Q1 16MHz, SW2 FSMSM, U2 ATMEGA328P-PU

Commit message: Redesigned Hardware
Parts:
- removed BT1: KEYSTONE_ELECTRONICS_3034KEYSTONE_ELECTRONICS_3034_0_0, Keystone Electronics - 3034:KEYSTONE_ELECTRONICS_3034KEYSTONE_ELECTRONICS_3034_0_0
- removed H1, H2: MOUNT-PAD-ROUND3.0, holes:MOUNT-PAD-ROUND3.0
- removed JP1, JP3: (no value), pinhead:PINHD-1X2
- removed JP2: (no value), pinhead:PINHD-1X4
- removed M2: WIRELESS-NRF24L01-PA-EXT, diy-modules:WIRELESS-NRF24L01-PA-EXT
- removed Q1: 16MHz, special:XTAL/S
- removed U$1: 1051620001A, Molex_micro_SD:1051620001A
- removed U2: ATMEGA328P-PU, Microcontroller:ATMEGA328P-PU
- added BT2: BAT-HLD-001, BAT-HLD-001:BAT-HLD-001
- added C5: .1 uF, rcl:C-USC0805
- added C6: 2.2 uF, rcl:C-USC0805
- added C7: 1 uF, rcl:C-USC0805
- added J1: MEM2067-02-180-00-A_REVB, MEM2067-02-180-00-A_REVB:MEM2067-02-180-00-A_REVB
- added J2, J3: 95501-2441, SamacSys_Parts:95501-2441
- added J4: PJ-102A, PJ-102A:PJ-102A
- added L2: 12 uH, rcl:L-USL1812
- added R10, R11, R12, R13, R14, R7, R8, R9: 10 K, rcl:R-US_R0805
- added SW1: FSM4JSMA, Switch:FSM4JSMA
- added U1: XB3-24Z8UM-J, XB3-24Z8UM-J:XB3-24Z8UM-J
- C1: value 22pF -> 8.2 pF; DATASHEET (none) -> https://www.mouser.com/datasheet/2/427/vjw1bcbascomseries-1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; MOUSER_NUM (none) -> 77-VJ0805A8R2BXXPBC; PRICE (none) -> .14; PRICE_50 (none) -> .1
- C2: value 22pF -> 1 uF; DATASHEET (none) -> https://www.mouser.com/datasheet/2/585/MLCC-1837944.pdf; MOUSER_NUM (none) -> 187-CL21B105KBFNNNG; PRICE (none) -> .11; PRICE_100 (none) -> .04
- C3: value .1uF -> 10 uF; DATASHEET (none) -> https://www.mouser.com/datasheet/2/585/MLCC-1837944.pdf; MOUSER_NUM (none) -> 187-CL21A106KOQNNNG; PRICE (none) -> .1; PRICE_10 (none) -> .044
- C4: value .1uF -> 22 uF; DATASHEET (none) -> https://www.mouser.com/datasheet/2/585/MLCC-1837944.pdf; MOUSER_NUM (none) -> 187-CL21A226MPQNNNE; PRICE (none) -> .18; PRICE_100 (none) -> .064
- IC1: value 4050D -> TPS560430X3FDBVR; device 40xx:4050D -> SamacSys_Parts:TPS560430X3FDBVR; DATASHEET (none) -> https://www.ti.com/lit/ds/symlink/tps560430.pdf?HQS=dis-mou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; MOUSER_NUM (none) -> 595-TPS560430X3FDBVR; PRICE (none) -> 1.19; PRICE_10 (none) -> 1.01
- IC2: value LP298XS -> DS3231SN; device adafruit:LP298XS -> SamacSys_Parts:DS3231SN; DATASHEET (none) -> https://www.mouser.com/datasheet/2/256/DS3231-1513891.pdf; MOUSER_NUM (none) -> 700-DS3231SN#T&R-; PRICE (none) -> 8.82; PRICE_50 (none) -> 7.37
- IC3: value DS3231/SO -> 4050D; device adafruit:DS3231/SO -> 40xx:4050D; DATASHEET (none) -> https://www.mouser.com/datasheet/2/916/74HC4050-1598370.pdf; MOUSER_NUM (none) -> 771-74HC4050D-T; PRICE (none) -> .51; PRICE_100 (none) -> 25.70
- LED1: value RED -> (none); device led:LEDCHIPLED_0805 -> led:LEDCHIP-LED0805; DATASHEET (none) -> https://dammedia.osram.info/media/resource/hires/osram-dam-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; MOUSER_NUM (none) -> 720-LGR971-KN-1; PRICE (none) -> .25; PRICE_100 (none) -> .058
- LED2: value GREEN -> (none); device led:LEDCHIPLED_0805 -> led:LEDCHIP-LED0805; DATASHEET (none) -> https://dammedia.osram.info/media/resource/hires/osram-dam-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; MOUSER_NUM (none) -> 720-LGR971-KN-1; PRICE (none) -> .25; PRICE_100 (none) -> .058
- LED3: value Yellow -> (none); device led:LEDCHIPLED_0805 -> led:LEDCHIP-LED0805; DATASHEET (none) -> https://dammedia.osram.info/media/resource/hires/osram-dam-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; MOUSER_NUM (none) -> 720-LGR971-KN-1; PRICE (none) -> .25; PRICE_100 (none) -> .058
- R1: value 1K -> 10 K; DATASHEET (none) -> https://www.mouser.com/datasheet/2/219/RK73H-1825326.pdf; MOUSER_NUM (none) -> 660-RK73H2ATTD1002F; PRICE (none) -> .1; PRICE_1000 (none) -> .006
- R2, R3: value 10K -> 10 K; DATASHEET (none) -> https://www.mouser.com/datasheet/2/219/RK73H-1825326.pdf; MOUSER_NUM (none) -> 660-RK73H2ATTD1002F; PRICE (none) -> .1; PRICE_1000 (none) -> .006
- R4: value 10K -> 160; DATASHEET (none) -> https://www.mouser.com/datasheet/2/219/RK73H-1825326.pdf; MOUSER_NUM (none) -> 660-RK73H2ATTD1600F; PRICE (none) -> .1; PRICE_100 (none) -> .014
- R5, R6: value 1K -> 160; DATASHEET (none) -> https://www.mouser.com/datasheet/2/219/RK73H-1825326.pdf; MOUSER_NUM (none) -> 660-RK73H2ATTD1600F; PRICE (none) -> .1; PRICE_100 (none) -> .014
- SW2: value FSMSM -> FSM4JSMA; device Switch:FSMSM -> Switch:FSM4JSMA; DATASHEET (none) -> https://www.mouser.com/datasheet/2/418/1/NG_CD_2-1437565-7_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; MOUSER_NUM (none) -> 506-FSM4JSMA; PRICE (none) -> .24; PRICE_100 (none) -> .197
Connections:
- removed net +5V: C3.1, IC2.EN, IC2.VIN, IC3.VCC, JP2.4, R2.2, R3.2, R4.2, U2.AVCC, U2.VCC
- removed net 32KHZ: IC3.32KHZ
- removed net CE: M2.CE, U2.(OC1A/PCINT1)PB1
- removed net CLK: IC1A.I, IC1D.I
- removed net CS: IC1C.I
- removed net CSN: M2.CSN, U2.(PCINT0/CLKO/ICP1)PB0
- removed net DI: IC1B.I
- removed net DO: U$1.DAT0
- removed net N$7: C1.1, Q1.1, U2.(PCINT7/XTAL2/TOSC2)PB7
- removed net SCK: M2.SCK, U2.(SCK/PCINT5)PB5
- removed net SQW: IC3.SQW/INT
- removed net VBAT: BT1.ANODE, IC3.VBAT
- removed net V_PACK: JP1.1
- new net !INT: IC2.!INT!/SQW, R3.1
- new net !SS: IC3C.I, U1.SPI_!SSEL!/DIO17
- new net ANEM_DIR: J2.2, R8.2
- new net ANEM_DIR/2: R8.1, R9.2, U1.AD2/DIO2
- new net ANEM_SPD: J2.3, R7.1, U1.AD3/DIO3
- new net N$13: R6.1, U1.ASSOCIATE/DIO5
- new net N$14: R11.1, SW1.1, SW1.2, U1.!RESET
- new net N$16: R10.2, SW2.3, SW2.4, U1.DIO12
- new net SCLK: IC3A.I, U1.SPI_CLK/DIO18
- new net VCC: C6.1, IC1.EN, IC1.VIN, J2.1, J4.1, R12.2, R7.2
- new net VCC/2: R12.1, R13.2, U1.AD0/DIO0
- net !RTC_RST: now also IC2.!RST, R14.1, U1.DOUT/DIO13; no longer IC3./RST
- net +3V3: now also C1.1, C2.1, C3.1, C7.1, IC2.VCC, IC3P.VDD, J1.VDD, J3.1, L2.1, R1.2, R11.2, R14.2, R2.2, R3.2, SW2.1, SW2.2, U1.VCC; no longer IC1P.VDD, IC2.VOUT, M2.VCC, U$1.VDD
- net GND: now also BT2.-, C6.2, C7.2, IC1.GND, IC2.N.C._1, IC2.N.C._2, IC2.N.C._3, IC2.N.C._4, IC2.N.C._5, IC2.N.C._6, IC2.N.C._7, IC2.N.C._8, IC3E.I, IC3F.I, IC3P.VSS, J1.SHIELD, J1.VSS, J2.4, J3.4, J4.2, R10.1, R13.1, R9.1, SW1.3, SW1.4, U1.GND; no longer BT1.CATHODE, IC1E.I, IC1F.I, IC1P.VSS, IC3.GND, JP1.2, JP2.3, JP3.2, M2.GND, SW2.2, U$1.GND, U$1.GND@1, U$1.GND@2, U$1.GND@3, U$1.VSS, U2.AREF, U2.GND, U2.GND1
- net MISO: now also J1.DAT0, U1.SPI_MISO/DIO15; no longer M2.MISO, U2.(MISO/PCINT4)PB4
- net MOSI: now also IC3B.I, U1.SPI_MOSI/DIO16; no longer M2.MOSI, U2.(MOSI/OC2A/PCINT3)PB3
- net N$1: now also LED2.A, R5.2; no longer IC1D.O, LED1.A
- net N$10: now also LED1.C, R4.1; no longer LED2.A, R5.1
- net N$11: now also IC3A.O, IC3D.I, J1.CLK; no longer LED3.A, R6.1
- net N$12: now also R5.1, U1.DIO4; no longer R6.2, U2.(PCINT22/OC0A/AIN0)PD6
- net N$2: now also IC3B.O, J1.CMD; no longer IC1A.O, U$1.CLK
- net N$3: now also C5.2, IC1.CB; no longer IC1C.O, R1.1, U$1.CD/DAT3
- net N$4: now also BT2.+, IC2.VBAT; no longer LED1.C, R1.2
- net N$5: now also C5.1, IC1.SW, L2.2; no longer IC1B.O, U$1.CMD
- net N$6: now also IC3C.O, J1.CD/DAT3, R4.2; no longer R2.1, SW2.1, U2.PC6(PCINT14/!RESET)
- net N$8: now also LED3.A, R6.2; no longer C2.1, Q1.2, U2.(PCINT6/XTAL1/TOSC1)PB6
- net N$9: now also IC3D.O, LED1.A; no longer R5.2, U2.(PCINT21/OC0B/T1)PD5
- net SCL: now also IC2.SCL, J3.2, R1.1, U1.AD1/DIO1; no longer IC3.SCL, JP2.2, R3.1, U2.PC5(ADC5/SCL/PCINT13)
- net SDA: now also IC2.SDA, J3.3, R2.1, U1.PWM1/DIO11; no longer IC3.SDA, JP2.1, R4.1, U2.PC4(ADC4/SDA/PCINT12)
Other:
- note added: "CO2_SENSOR"
- note added: "MICROSD"
- note added: "Mesh network CO2 sensor network node. Powered by 5 volt power jack. Uses XBEE 3 pro mmt for processing and radio communications. Node contains an RTC clock and MicroSD read/write capabilities."
- note added: "POWER"
- note added: "RTC"
- note added: "WIND_SENSOR"
- note added: "XBEE"
- note added: "v0.1"
- note removed: "Sensor network node powered by an ATMEGA328. Collects data with a C02 sensor each second by utilizing an RTC. Stores data on a microSD card, and syncronizes periodically with a central network hub."
- moved on the sheet: C1, C2, C3, C4, LED1, LED2, LED3, R1, R2, R3, R4, R5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
